File: HW2/sgd710_pic32_pcb/sgd710_pic32_sch.sch (EAGLE design)
At the start: 22 parts, among them J1 USB-MB-H

Commit message: 4/17/18
Parts:
- U$3: value MCP1702T -> MCP1702
- U$9: value OSC -> 8MHz
Connections:
- net +3V3: now also R3.1, R4.1; no longer C1.2, U$1.27.AVSS
- net B4/USER: now also U$5.2; no longer U$4.2
- net GND: now also C1.2, U$1.27.AVSS; no longer R3.1, R4.1
- net MCLR: now also U$4.2; no longer U$5.2
